File: PCB/version1.kicad_pcb (KiCad board)
At the start: 2 copper layers, 395 x 135 mm, 213 parts, among them J1 USB_C_Receptacle_USB2.0_16P, SW1 SW_SPST, SW2 SW_SPST, SW3 RotaryEncoder_Switch, U1 STM32F072CBTx, U2 XC6206PxxxMR

Commit message: Updated PCB files
Parts:
- added J2: Conn_01x04_Pin, Connector_PinHeader_2.54mm:PinHeader_1x04_P2.54mm_Horizontal, F.Cu at (379.3, 109.6)
Routing:
- net SWDIO: track 0.00 -> 35.6 mm, vias 0 -> 1
- net SWCLK: track 0.00 -> 30.0 mm, vias 0 -> 1
- net +3V3: track 52.8 -> 68.8 mm
- net GND: track 43.1 -> 44.8 mm, vias 25 -> 26
